File: 4x3Matrix/kicad/3x4Matrix_3x072.kicad_pcb (KiCad board)
At the start: 2 copper layers, 99.4 x 49.5 mm, 59 parts, among them M1 AudioJack, M2 AudioJack, M3 AudioJack, M4 AudioJack, U1 TL072_SMD, U2 TL072_SMD, U3 TL072_SMD

Commit message: Corrections made to ground planes, trace widths, etc. after visual checks of printout
Parts:
- removed MCC34: AudioJack, Connector_Audio:Jack_3.5mm_QingPu_WQP-PJ398SM_Vertical_CircularHoles
- added OUTC1: AudioJack, Connector_Audio:Jack_3.5mm_QingPu_WQP-PJ398SM_Vertical_CircularHoles, F.Cu at (193.4, 93.2)
- moved C3 0.20 mm to (158.2, 94.1)
- moved C4 0.20 mm to (158.2, 92.0)
- renumbered A1 to A_1, A2 to A_2, A3 to A_3, A4 to A_4, B1 to B_1, B2 to B_2, B3 to B_3, B4 to B_4, C-1-34 to C_1, C-2 to C_2, C-3 to C_3, C-4 to C_4, D3 to D1, D4 to D2, M1 to IN1, M2 to IN2, M3 to IN3, M4 to IN4, MAA34 to OUTA1, MB34 to OUTB1
Connections:
- A_1 pad : (no net) -> GND
- A_2 pad : (no net) -> GND
- A_3 pad : (no net) -> GND
- A_4 pad : (no net) -> GND
- B_1 pad : (no net) -> GND
- B_2 pad : (no net) -> GND
- B_3 pad : (no net) -> GND
- B_4 pad : (no net) -> GND
- C_1 pad : (no net) -> GND
- C_2 pad : (no net) -> GND
- C_3 pad : (no net) -> GND
- C_4 pad : (no net) -> GND
Routing:
- net /C-11: track 70.9 -> 71.7 mm
- net /N$12: track 72.3 -> 73.1 mm
- net /N$29: track 61.5 -> 60.7 mm
- net /N$26: track 89.7 -> 89.0 mm
Other:
- net class Default: trace_width 0.3 -> 0.35
- net class Power added: clearance 0.2, trace_width 0.5, via_dia 1, via_drill 0.5
- board text added: "-12"
- board text added: "Remake of Pusherman's 3x4Matrix 3x072 edition KiCad layout v0.2 by zero.emission"
