File: 4x3Matrix/kicad/3x4Matrix_3x072.sch (KiCad schematic (older format))
At the start: 54 parts, among them M1 AudioJack, M2 AudioJack, M3 AudioJack, M4 AudioJack, U1 TL074_SMD, U2 TL072_SMD

Commit message: All library parts replaced by default Kicad, new version created which uses 3 TL072 instead of TL072 + TL074 to eliminate crosstalk
Parts:
- removed unit 3 of U1
- removed unit 4 of U1
- removed unit 5 of U1
- added C3, C4: 100nF, Capacitor_SMD:C_0805_2012Metric, symbol Device:C
- added unit 3 of U1
- added U2: TL072_SMD, Package_SO:SOIC-8_3.9x4.9mm_P1.27mm, symbol Amplifier_Operational:TL072
- U1: value TL074_SMD -> TL072_SMD; footprint Package_SO:SOIC-14_3.9x8.7mm_P1.27mm -> Package_SO:SOIC-8_3.9x4.9mm_P1.27mm; symbol Amplifier_Operational:TL074 -> Amplifier_Operational:TL072
- renumbered C8 to C1, C7 to C2, C1 to C5, C11 to C6, C10 to C7, C9 to C8, U2 to U3
Connections:
- wire segments 212 -> 218
Changed lines of the file:
@@
 $EndComp
 $Comp
-L Device:C C1
+L Device:C C5
 U 1 1 5EFF2ECB
 P 5450 6500
-F 0 "C1" H 5400 6150 70  0000 L BNN
+F 0 "C5" H 5400 6150 70  0000 L BNN
 F 1 "100nF" H 5400 6000 70  0000 L BNN
 F 2 "Capacitor_SMD:C_0805_2012Metric" H 5440 6290 65  0001 L TNN
@@
 $EndComp
 $Comp
-L Device:CP C7
+L Device:CP C2
 U 1 1 5EFF2F93
 P 1950 6200
-F 0 "C7" H 1700 6250 70  0000 L BNN
+F 0 "C2" H 1700 6250 70  0000 L BNN
 F 1 "10uF" H 1650 6000 70  0000 L BNN
 F 2 "Capacitor_THT:CP_Radial_D5.0mm_P2.50mm" H 1940 5990 65  0001 L TNN
@@
 $EndComp
 $Comp
-L Device:CP C8
+L Device:CP C1
 U 1 1 5EFF305B
 P 1950 6600
-F 0 "C8" H 1750 6650 70  0000 L BNN
+F 0 "C1" H 1750 6650 70  0000 L BNN
 F 1 "10uF" H 1650 6450 70  0000 L BNN
 F 2 "Capacitor_THT:CP_Radial_D5.0mm_P2.50mm" H 1940 6390 65  0001 L TNN
@@
 $EndComp
 $Comp
-L Device:C C9
+L Device:C C8
 U 1 1 5EFF3123
 P 4850 6100
-F 0 "C9" H 4750 6500 70  0000 L BNN
+F 0 "C8" H 4750 6500 70  0000 L BNN
 F 1 "100nF" H 4750 6350 70  0000 L BNN
 F 2 "Capacitor_SMD:C_0805_2012Metric" H 4840 5890 65  0001 L TNN
@@
 $EndComp
 $Comp
-L Device:C C10
+L Device:C C7
 U 1 1 5EFF31EB
 P 4850 6600
-F 0 "C10" H 4800 6350 70  0000 L BNN
+F 0 "C7" H 4800 6350 70  0000 L BNN
 F 1 "100nF" H 4800 6200 70  0000 L BNN
 F 2 "Capacitor_SMD:C_0805_2012Metric" H 4840 6390 65  0001 L TNN
@@
 $EndComp
 $Comp
-L Device:C C11
+L Device:C C6
 U 1 1 5EFF32B3
 P 5450 6100
-F 0 "C11" H 5300 6500 70  0000 L BNN
+F 0 "C6" H 5300 6500 70  0000 L BNN
 F 1 "100nF" H 5300 6350 70  0000 L BNN
 F 2 "Capacitor_SMD:C_0805_2012Metric" H 5440 5890 65  0001 L TNN
@@
 	4850 6750 4450 6750
 Wire Wire Line
-	4450 6750 4150 6750
-Wire Wire Line
 	3950 6650 3550 6650
 Wire Wire Line
@@
 	3950 6250 3950 6150
 Wire Wire Line
-	3950 6150 4150 6150
-Wire Wire Line
-	4150 6150 4450 6150
-Wire Wire Line
 	4450 6150 4650 6150
 Wire Wire Line
@@
 Connection ~ 4850 5950
 Connection ~ 3950 6150
-Connection ~ 4150 6150
 Connection ~ 4450 6150
 Wire Wire Line
@@
 Connection ~ 5450 6350
 $Comp
-L Amplifier_Operational:TL072 U2
+L Amplifier_Operational:TL072 U3
 U 3 1 5EFF5A8B
 P 4550 6450
-F 0 "U2" H 4540 6440 65  0001 L TNN
+F 0 "U3" H 4540 6440 65  0001 L TNN
 F 1 "TL072_SMD" H 4540 6340 65  0001 L TNN
 F 2 "Package_SO:SOIC-8_3.9x4.9mm_P1.27mm" H 4540 6240 65  0001 L TNN
@@
 $EndComp
 $Comp
-L Amplifier_Operational:TL072 U2
+L Amplifier_Operational:TL072 U3
 U 1 1 5EFF59C3
 P 6450 4450
-F 0 "U2" H 6549 4575 70  0000 L BNN
+F 0 "U3" H 6549 4575 70  0000 L BNN
 F 1 "TL072_SMD" H 6550 4250 70  0000 L BNN
 F 2 "Package_SO:SOIC-8_3.9x4.9mm_P1.27mm" H 6440 4240 65  0001 L TNN
@@
 $EndComp
 $Comp
-L Amplifier_Operational:TL072 U2
+L Amplifier_Operational:TL072 U3
 U 2 1 5EFF5A27
 P 7550 4450
-F 0 "U2" H 7649 4575 70  0000 L BNN
+F 0 "U3" H 7649 4575 70  0000 L BNN
 F 1 "TL072_SMD" H 7650 4250 70  0000 L BNN
 F 2 "Package_SO:SOIC-8_3.9x4.9mm_P1.27mm" H 7540 4240 65  0001 L TNN
 F 3 "" H 7550 4450 50  0001 C CNN
 	2    7550 4450
-	1    0    0    1
-$EndComp
-$Comp
-L Amplifier_Operational:TL074 U1
-U 5 1 5EFF58FB
-P 4250 6450
-F 0 "U1" H 4240 6440 65  0001 L TNN
-F 1 "TL074_SMD" H 4240 6340 65  0001 L TNN
-F 2 "Package_SO:SOIC-14_3.9x8.7mm_P1.27mm" H 4240 6240 65  0001 L TNN
-F 3 "" H 4250 6450 50  0001 C CNN
-	5    4250 6450
-	1    0    0    -1
-$EndComp
-$Comp
-L Amplifier_Operational:TL074 U1
-U 4 1 5EFF5897
-P 7550 2950
-F 0 "U1" H 7649 3075 70  0000 L BNN
-F 1 "TL074_SMD" H 7650 2750 70  0000 L BNN
-F 2 "Package_SO:SOIC-14_3.9x8.7mm_P1.27mm" H 7540 2740 65  0001 L TNN
-F 3 "" H 7550 2950 50  0001 C CNN
-	4    7550 2950
-	1    0    0    1
-$EndComp
-$Comp
-L Amplifier_Operational:TL074 U1
-U 2 1 5EFF57CF
-P 7550 1450
-F 0 "U1" H 7649 1575 70  0000 L BNN
-F 1 "TL074_SMD" H 7650 1250 70  0000 L BNN
-F 2 "Package_SO:SOIC-14_3.9x8.7mm_P1.27mm" H 7540 1240 65  0001 L TNN
-F 3 "" H 7550 1450 50  0001 C CNN
-	2    7550 1450
-	1    0    0    1
-$EndComp
-$Comp
-L Amplifier_Operational:TL074 U1
-U 1 1 5EFF576B
-P 6450 1450
-F 0 "U1" H 6549 1575 70  0000 L BNN
-F 1 "TL074_SMD" H 6550 1250 70  0000 L BNN
-F 2 "Package_SO:SOIC-14_3.9x8.7mm_P1.27mm" H 6440 1240 65  0001 L TNN
-F 3 "" H 6450 1450 50  0001 C CNN
-	1    6450 1450
-	1    0    0    1
-$EndComp
-$Comp
-L Amplifier_Operational:TL074 U1
-U 3 1 5EFF5833
-P 6450 2950
-F 0 "U1" H 6549 3075 70  0000 L BNN
-F 1 "TL074_SMD" H 6550 2750 70  0000 L BNN
-F 2 "Package_SO:SOIC-14_3.9x8.7mm_P1.27mm" H 6440 2740 65  0001 L TNN
-F 3 "" H 6450 2950 50  0001 C CNN
-	3    6450 2950
 	1    0    0    1
 $EndComp
@@
 Wire Wire Line
 	3550 6250 3950 6250
+Connection ~ 3950 6750
+Wire Wire Line
+	3950 6750 3950 6650
+Wire Wire Line
+	1950 6750 1950 7150
+Wire Wire Line
+	1950 7150 3950 7150
+$Comp
+L Amplifier_Operational:TL072 U1
+U 1 1 5EFF576B
+P 6450 1450
+F 0 "U1" H 6549 1575 70  0000 L BNN
+F 1 "TL072_SMD" H 6550 1250 70  0000 L BNN
+F 2 "Package_SO:SOIC-8_3.9x4.9mm_P1.27mm" H 6440 1240 65  0001 L TNN
+F 3 "http://www.ti.com/lit/ds/symlink/tl071.pdf" H 6450 1450 50  0001 C CNN
+	1    6450 1450
+	1    0    0    1
+$EndComp
+$Comp
+L Amplifier_Operational:TL072 U1
+U 2 1 5EFF57CF
+P 7550 1450
+F 0 "U1" H 7649 1575 70  0000 L BNN
+F 1 "TL072_SMD" H 7650 1250 70  0000 L BNN
+F 2 "Package_SO:SOIC-8_3.9x4.9mm_P1.27mm" H 7540 1240 65  0001 L TNN
+F 3 "http://www.ti.com/lit/ds/symlink/tl071.pdf" H 7550 1450 50  0001 C CNN
+	2    7550 1450
+	1    0    0    1
+$EndComp
 Wire Wire Line
 	3950 6750 4150 6750
-Connection ~ 3950 6750
-Wire Wire Line
-	3950 6750 3950 6650
+Wire Wire Line
+	3950 6150 4150 6150
+$Comp
+L Amplifier_Operational:TL072 U1
+U 3 1 5F181DA9
+P 4250 6450
+F 0 "U1" H 4208 6496 50  0001 L CNN
+F 1 "TL072_SMD" H 4208 6405 50  0001 L CNN
+F 2 "Package_SO:SOIC-8_3.9x4.9mm_P1.27mm" H 4250 6450 50  0001 C CNN
+F 3 "http://www.ti.com/lit/ds/symlink/tl071.pdf" H 4250 6450 50  0001 C CNN
+	3    4250 6450
+	1    0    0    -1
+$EndComp
 Connection ~ 4150 6750
 Wire Wire Line
-	1950 6750 1950 7150
-Wire Wire Line
-	1950 7150 3950 7150
+	4150 6750 4300 6750
+Connection ~ 4150 6150
+Wire Wire Line
+	4150 6150 4300 6150
+$Comp
+L Amplifier_Operational:TL072 U2
+U 1 1 5F1BB2B0
+P 6450 2950
+F 0 "U2" H 6549 3075 70  0000 L BNN
+F 1 "TL072_SMD" H 6550 2750 70  0000 L BNN
+F 2 "Package_SO:SOIC-8_3.9x4.9mm_P1.27mm" H 6440 2740 65  0001 L TNN
+F 3 "http://www.ti.com/lit/ds/symlink/tl071.pdf" H 6450 2950 50  0001 C CNN
+	1    6450 2950
+	1    0    0    1
+$EndComp
+$Comp
+L Amplifier_Operational:TL072 U2
+U 2 1 5F1C17C2
+P 7550 2950
+F 0 "U2" H 7649 3075 70  0000 L BNN
+F 1 "TL072_SMD" H 7650 2750 70  0000 L BNN
+F 2 "Package_SO:SOIC-8_3.9x4.9mm_P1.27mm" H 7540 2740 65  0001 L TNN
+F 3 "http://www.ti.com/lit/ds/symlink/tl071.pdf" H 7550 2950 50  0001 C CNN
+	2    7550 2950
+	1    0    0    1
+$EndComp
+$Comp
+L Amplifier_Operational:TL072 U2
+U 3 1 5F1D1498
+P 4400 6450
+F 0 "U2" H 4358 6496 50  0001 L CNN
+F 1 "TL072_SMD" H 4358 6405 50  0001 L CNN
+F 2 "Package_SO:SOIC-8_3.9x4.9mm_P1.27mm" H 4400 6450 50  0001 C CNN
+F 3 "http://www.ti.com/lit/ds/symlink/tl071.pdf" H 4400 6450 50  0001 C CNN
+	3    4400 6450
+	1    0    0    -1
+$EndComp
+Connection ~ 4300 6750
+Wire Wire Line
+	4300 6750 4450 6750
+Connection ~ 4300 6150
+Wire Wire Line
+	4300 6150 4450 6150
+$Comp
+L Device:C C4
+U 1 1 5F1A823F
+P 6150 6100
+F 0 "C4" H 6000 6500 70  0000 L BNN
+F 1 "100nF" H 6000 6350 70  0000 L BNN
+F 2 "Capacitor_SMD:C_0805_2012Metric" H 6140 5890 65  0001 L TNN
+F 3 "" H 6150 6100 50  0001 C CNN
+	1    6150 6100
+	1    0    0    -1
+$EndComp
+$Comp
+L Device:C C3
+U 1 1 5F1A8B92
+P 6150 6600
+F 0 "C3" H 6100 6250 70  0000 L BNN
+F 1 "100nF" H 6100 6100 70  0000 L BNN
+F 2 "Capacitor_SMD:C_0805_2012Metric" H 6140 6390 65  0001 L TNN
+F 3 "" H 6150 6600 50  0001 C CNN
+	1    6150 6600
+	1    0    0    -1
+$EndComp
+Wire Wire Line
+	5450 6750 6150 6750
+Connection ~ 5450 6750
+Wire Wire Line
+	5450 5950 6150 5950
+Connection ~ 5450 5950
+Wire Wire Line
+	6150 6250 6150 6350
+$Comp
+L power:GND #GND?
+U 1 1 5F1DDE6D
+P 6150 6350
+F 0 "#GND?" V 6150 5750 70  0000 L BNN
+F 1 "GND" V 6250 6000 70  0000 L BNN
+F 2 "" H 6150 6350 60  0001 C CNN
+F 3 "" H 6150 6350 60  0001 C CNN
+	1    6150 6350
+	0    -1   -1   0
+$EndComp
+Connection ~ 6150 6350
+Wire Wire Line
+	6150 6350 6150 6450
 $EndSCHEMATC

Commit message: Corrections made to ground planes, trace widths, etc. after visual checks of printout
Parts:
- renumbered A1 to A_1, A2 to A_2, A3 to A_3, A4 to A_4, B1 to B_1, B2 to B_2, B3 to B_3, B4 to B_4, C-1-34 to C_1, C-2 to C_2, C-3 to C_3, C-4 to C_4, D3 to D1, D4 to D2, M1 to IN1, M2 to IN2, M3 to IN3, M4 to IN4, MAA34 to OUTA1, MB34 to OUTB1, MCC34 to OUTC1
Changed lines of the file:
@@
 $EndDescr
 $Comp
-L Device:R_POT A1
+L Device:R_POT A_1
 U 1 1 5EFF2507
 P 4150 4750
-F 0 "A1" V 3950 4651 70  0000 L BNN
+F 0 "A_1" V 3950 4651 70  0000 L BNN
 F 1 "A100K" V 4050 4650 70  0000 L BNN
 F 2 "Potentiometer_THT:Potentiometer_Alpha_RD901F-40-00D_Single_Vertical" H 4140 4540 65  0001 L TNN
@@
 $EndComp
 $Comp
-L Device:R_POT A2
+L Device:R_POT A_2
 U 1 1 5EFF25CF
 P 4150 3850
-F 0 "A2" V 3950 3751 70  0000 L BNN
+F 0 "A_2" V 3950 3751 70  0000 L BNN
 F 1 "A100K" V 4050 3750 70  0000 L BNN
 F 2 "Potentiometer_THT:Potentiometer_Alpha_RD901F-40-00D_Single_Vertical" H 4140 3640 65  0001 L TNN
@@
 $EndComp
 $Comp
-L Device:R_POT A3
+L Device:R_POT A_3
 U 1 1 5EFF2697
 P 4150 2950
-F 0 "A3" V 3950 2851 70  0000 L BNN
+F 0 "A_3" V 3950 2851 70  0000 L BNN
 F 1 "A100K" V 4050 2850 70  0000 L BNN
 F 2 "Potentiometer_THT:Potentiometer_Alpha_RD901F-40-00D_Single_Vertical" H 4140 2740 65  0001 L TNN
@@
 $EndComp
 $Comp
-L Device:R_POT A4
+L Device:R_POT A_4
 U 1 1 5EFF275F
 P 4150 1950
-F 0 "A4" V 3950 1851 70  0000 L BNN
+F 0 "A_4" V 3950 1851 70  0000 L BNN
 F 1 "A100K" V 4050 1850 70  0000 L BNN
 F 2 "Potentiometer_THT:Potentiometer_Alpha_RD901F-40-00D_Single_Vertical" H 4140 1740 65  0001 L TNN
@@
 $EndComp
 $Comp
-L Device:R_POT B1
+L Device:R_POT B_1
 U 1 1 5EFF2827
 P 3150 4750
-F 0 "B1" V 2950 4651 70  0000 L BNN
+F 0 "B_1" V 2950 4651 70  0000 L BNN
 F 1 "A100K" V 3050 4650 70  0000 L BNN
 F 2 "Potentiometer_THT:Potentiometer_Alpha_RD901F-40-00D_Single_Vertical" H 3140 4540 65  0001 L TNN
@@
 $EndComp
 $Comp
-L Device:R_POT B2
+L Device:R_POT B_2
 U 1 1 5EFF28EF
 P 3150 3850
-F 0 "B2" V 2950 3751 70  0000 L BNN
+F 0 "B_2" V 2950 3751 70  0000 L BNN
 F 1 "A100K" V 3050 3750 70  0000 L BNN
 F 2 "Potentiometer_THT:Potentiometer_Alpha_RD901F-40-00D_Single_Vertical" H 3140 3640 65  0001 L TNN
@@
 $EndComp
 $Comp
-L Device:R_POT B3
+L Device:R_POT B_3
 U 1 1 5EFF29B7
 P 3150 2950
-F 0 "B3" V 2950 2851 70  0000 L BNN
+F 0 "B_3" V 2950 2851 70  0000 L BNN
 F 1 "A100K" V 3050 2850 70  0000 L BNN
 F 2 "Potentiometer_THT:Potentiometer_Alpha_RD901F-40-00D_Single_Vertical" H 3140 2740 65  0001 L TNN
@@
 $EndComp
 $Comp
-L Device:R_POT B4
+L Device:R_POT B_4
 U 1 1 5EFF2A7F
 P 3150 1950
-F 0 "B4" V 2950 1851 70  0000 L BNN
+F 0 "B_4" V 2950 1851 70  0000 L BNN
 F 1 "A100K" V 3050 1850 70  0000 L BNN
 F 2 "Potentiometer_THT:Potentiometer_Alpha_RD901F-40-00D_Single_Vertical" H 3140 1740 65  0001 L TNN
@@
 $EndComp
 $Comp
-L Device:R_POT C-1-34
+L Device:R_POT C_1
 U 1 1 5EFF2BAB
 P 2150 4750
-F 0 "C-1-34" V 1950 4651 70  0000 L BNN
+F 0 "C_1" V 1950 4651 70  0000 L BNN
 F 1 "A100K" V 2050 4650 70  0000 L BNN
 F 2 "Potentiometer_THT:Potentiometer_Alpha_RD901F-40-00D_Single_Vertical" H 2140 4540 65  0001 L TNN
@@
 $EndComp
 $Comp
-L Device:R_POT C-2
+L Device:R_POT C_2
 U 1 1 5EFF2C73
 P 2150 3850
-F 0 "C-2" V 1950 3751 70  0000 L BNN
+F 0 "C_2" V 1950 3751 70  0000 L BNN
 F 1 "A100K" V 2050 3750 70  0000 L BNN
 F 2 "Potentiometer_THT:Potentiometer_Alpha_RD901F-40-00D_Single_Vertical" H 2140 3640 65  0001 L TNN
@@
 $EndComp
 $Comp
-L Device:R_POT C-3
+L Device:R_POT C_3
 U 1 1 5EFF2D3B
 P 2150 2950
-F 0 "C-3" V 1950 2851 70  0000 L BNN
+F 0 "C_3" V 1950 2851 70  0000 L BNN
 F 1 "A100K" V 2050 2850 70  0000 L BNN
 F 2 "Potentiometer_THT:Potentiometer_Alpha_RD901F-40-00D_Single_Vertical" H 2140 2740 65  0001 L TNN
@@
 $EndComp
 $Comp
-L Device:R_POT C-4
+L Device:R_POT C_4
 U 1 1 5EFF2E03
 P 2150 1950
-F 0 "C-4" V 1950 1851 70  0000 L BNN
+F 0 "C_4" V 1950 1851 70  0000 L BNN
 F 1 "A100K" V 2050 1850 70  0000 L BNN
 F 2 "Potentiometer_THT:Potentiometer_Alpha_RD901F-40-00D_Single_Vertical" H 2140 1740 65  0001 L TNN
@@
 $EndComp
 $Comp
-L Device:D D4
+L Device:D D2
 U 1 1 5EFF3443
 P 3400 6650
-F 0 "D4" H 3500 6669 70  0000 L BNN
+F 0 "D2" H 3500 6669 70  0000 L BNN
 F 1 "1N4004" H 3500 6559 70  0000 L BNN
 F 2 "Diode_THT:D_DO-41_SOD81_P10.16mm_Horizontal" H 3390 6440 65  0001 L TNN
@@
 $EndComp
 $Comp
-L Connector:AudioJack2_SwitchT M1
+L Connector:AudioJack2_SwitchT IN1
 U 1 1 5EFF3E6B
 P 1600 4350
-F 0 "M1" H 1500 4510 70  0000 L BNN
+F 0 "IN1" H 1500 4510 70  0000 L BNN
 F 1 "AudioJack" H 1590 4240 65  0001 L TNN
 F 2 "Connector_Audio:Jack_3.5mm_QingPu_WQP-PJ398SM_Vertical_CircularHoles" H 1590 4140 65  0001 L TNN
@@
 $EndComp
 $Comp
-L Connector:AudioJack2_SwitchT M2
+L Connector:AudioJack2_SwitchT IN2
 U 1 1 5EFF3F33
 P 1600 3450
-F 0 "M2" H 1500 3610 70  0000 L BNN
+F 0 "IN2" H 1500 3610 70  0000 L BNN
 F 1 "AudioJack" H 1590 3340 65  0001 L TNN
 F 2 "Connector_Audio:Jack_3.5mm_QingPu_WQP-PJ398SM_Vertical_CircularHoles" H 1590 3240 65  0001 L TNN
@@
 $EndComp
 $Comp
-L Connector:AudioJack2_SwitchT M3
+L Connector:AudioJack2_SwitchT IN3
 U 1 1 5EFF3FFB
 P 1600 2550
-F 0 "M3" H 1500 2710 70  0000 L BNN
+F 0 "IN3" H 1500 2710 70  0000 L BNN
 F 1 "AudioJack" H 1590 2440 65  0001 L TNN
 F 2 "Connector_Audio:Jack_3.5mm_QingPu_WQP-PJ398SM_Vertical_CircularHoles" H 1590 2340 65  0001 L TNN
@@
 $EndComp
 $Comp
-L Connector:AudioJack2_SwitchT M4
+L Connector:AudioJack2_SwitchT IN4
 U 1 1 5EFF40C3
 P 1550 1550
-F 0 "M4" H 1450 1710 70  0000 L BNN
+F 0 "IN4" H 1450 1710 70  0000 L BNN
 F 1 "AudioJack" H 1540 1440 65  0001 L TNN
 F 2 "Connector_Audio:Jack_3.5mm_QingPu_WQP-PJ398SM_Vertical_CircularHoles" H 1540 1340 65  0001 L TNN
@@
 $EndComp
 $Comp
-L Connector:AudioJack2_SwitchT MAA34
+L Connector:AudioJack2_SwitchT OUTA1
 U 1 1 5EFF418B
 P 9650 4550
-F 0 "MAA34" H 9500 4250 70  0000 L BNN
+F 0 "OUTA1" H 9500 4250 70  0000 L BNN
 F 1 "AudioJack" H 9640 4440 65  0001 L TNN
 F 2 "Connector_Audio:Jack_3.5mm_QingPu_WQP-PJ398SM_Vertical_CircularHoles" H 9640 4340 65  0001 L TNN
@@
 $EndComp
 $Comp
-L Connector:AudioJack2_SwitchT MB34
+L Connector:AudioJack2_SwitchT OUTB1
 U 1 1 5EFF4253
 P 9550 3050
-F 0 "MB34" H 9400 2700 70  0000 L BNN
+F 0 "OUTB1" H 9400 2700 70  0000 L BNN
 F 1 "AudioJack" H 9540 2940 65  0001 L TNN
 F 2 "Connector_Audio:Jack_3.5mm_QingPu_WQP-PJ398SM_Vertical_CircularHoles" H 9540 2840 65  0001 L TNN
@@
 $EndComp
 $Comp
-L Connector:AudioJack2_SwitchT MCC34
+L Connector:AudioJack2_SwitchT OUTC1
 U 1 1 5EFF431B
 P 9450 1550
-F 0 "MCC34" H 9250 1200 70  0000 L BNN
+F 0 "OUTC1" H 9250 1200 70  0000 L BNN
 F 1 "AudioJack" H 9440 1440 65  0001 L TNN
 F 2 "Connector_Audio:Jack_3.5mm_QingPu_WQP-PJ398SM_Vertical_CircularHoles" H 9440 1340 65  0001 L TNN
@@
 	9000 4450 9350 4450
 $Comp
-L Device:D D3
+L Device:D D1
 U 1 1 5EFF337B
 P 3400 6250
-F 0 "D3" H 3500 6268 70  0000 L BNN
+F 0 "D1" H 3500 6268 70  0000 L BNN
 F 1 "1N4004" H 3500 6159 70  0000 L BNN
 F 2 "Diode_THT:D_DO-41_SOD81_P10.16mm_Horizontal" H 3390 6040 65  0001 L TNN
